File: KiCAD/APEDSK-AU.sch (KiCad schematic (older format))
At the start: 26 parts, among them J1 240-44-44Pins, P1 Power, P2 Analog, P3 Digital, P4 Digital, U1 74LS245, U2 74LS541, U3 74LS541, U4 74LS138, U5 74HC595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

Commit message: Latest files
Latest files
Parts:
- R1: value 100R -> 68R
- R2, R3, R4, R5: value 10K -> 5.1K
Connections:
- net A10: now also U2.7 (A5); no longer U3.4 (A2)
- net A11: now also U2.6 (A4); no longer U3.5 (A3)
- net A12: now also U2.5 (A3); no longer U3.6 (A4)
- net A15: now also U2.2 (A0); no longer U3.7 (A5)
- net A3: now also U3.6 (A4); no longer U2.5 (A3)
- net A4: now also U3.5 (A3); no longer U2.6 (A4)
- net A5: now also U3.4 (A2); no longer U2.7 (A5)
- net A6: now also U3.3 (A1); no longer U2.8 (A6)
- net A7: now also U3.2 (A0); no longer U2.9 (A7)
- net A8: now also U2.9 (A7); no longer U3.2 (A0)
- net A9: now also U2.8 (A6); no longer U3.3 (A1)
- net AD_A0: now also U4.6 (E3)
- net CLOCK: now also P2.6 (Pin_6); no longer P2.3 (Pin_3)
- net D0: now also U1.11 (B7); no longer U1.18 (B0)
- net D1: now also U1.12 (B6); no longer U1.17 (B1)
- net D2: now also U1.13 (B5); no longer U1.16 (B2)
- net D3: now also U1.14 (B4); no longer U1.15 (B3)
- net D4: now also U1.15 (B3); no longer U1.14 (B4)
- net D5: now also U1.16 (B2); no longer U1.13 (B5)
- net D6: now also U1.17 (B1); no longer U1.12 (B6)
- net D7: now also U1.18 (B0); no longer U1.11 (B7)
- net DS: now also P2.4 (Pin_4); no longer P2.1 (Pin_1)
- net GND: now also U3.7 (A5)
- net LATCH: now also P2.5 (Pin_5); no longer P2.2 (Pin_2)
- net ~AD_WE: now also P2.3 (Pin_3), U4.4 (E1); no longer P2.6 (Pin_6), U4.5 (E2)
- net ~TIBUF: now also P2.2 (Pin_2); no longer P2.5 (Pin_5)
- net A13: now reaches J1.15 (Pin_15)
- net A13: now also U2.4 (A2)
- net A14: now reaches J1.16 (Pin_16)
- net A14: now also U2.3 (A1)
- net A0: no longer names the net of J1.31 (Pin_31)
- net A0: no longer U2.2 (A0)
- net A1: no longer names the net of J1.30 (Pin_30)
- net A1: no longer U2.3 (A1)
- net A2: no longer names the net of J1.20 (Pin_20)
- net A2: no longer U2.4 (A2)
- net AD_A15: no longer names the net of U3.13 (Y5)
- net AD_A15: no longer U4.6 (E3)
- net ~AD_MBE renamed ~AD_CE
- net ~AD_CE: now also P2.1 (Pin_1), U4.5 (E2); no longer P2.4 (Pin_4), U4.4 (E1)
- no-connect marks 38 -> 41
Other:
- moved on the sheet: D1, R3, R4, R5, R6
