File: KiCAD/APEDSK-AU.kicad_pcb (KiCad board)
At the start: 4 copper layers, 71.1 x 68.6 mm, 26 parts, among them J1 240-44-44Pins, P1 Power, P2 Analog, P3 Digital, P4 Digital, U1 74LS245, U2 74LS541, U3 74LS541, U4 74LS138, U5 74HC595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

Commit message: R1, MBE
Parts:
- removed the R2 at (168.1, 89.5)
- renumbered R3 to R2, R4 to R3, R5 to R4, R6 to R5
Connections:
- U1 pad 19: /~AD_WE -> /CE_245
- U3 pad 13: Net-(U3-Pad13) -> /CE_245
- U3 pad 7: GND -> /~MBE
Routing:
- net /CE_245: track 0.00 -> 78.6 mm
- net /~AD_WE: track 140.1 -> 97.6 mm
- net /~MBE: track 68.5 -> 71.1 mm

Commit message: update
Parts:
- removed the R1 at (168.1, 81.9)
- added D2: 1N5711, Diode_THT:D_A-405_P5.08mm_Vertical_AnodeUp, F.Cu at (168.1, 85.7)
- renumbered R2 to R1, R3 to R2, R4 to R3, R5 to R4
Connections:
- net /TI_INT renamed /~TI_INT
- P2 pad 4: /DS -> /CLOCK
- P2 pad 6: /CLOCK -> /DS
- P4 pad 5: /AD_D1 -> /~AR_BUF
- P4 pad 7: /AD_D0 -> /AD_D1
- P4 pad 8: /~AR_BUF -> /AD_D0
Routing:
- net /~AR_BUF: track 112.3 -> 94.0 mm
- net /~AD_WE: track 97.6 -> 91.5 mm
- net /CLOCK: track 74.9 -> 68.9 mm
- net /READY: track 113.7 -> 110.1 mm
- net /AD_D0: track 134.7 -> 137.9 mm
- net /~TIBUF: track 79.3 -> 81.8 mm
- net /AD_D1: track 142.4 -> 141.7 mm
Other:
- board text added: "(c) 2020 Jochen Buur"
- board text added: "APEDSK99 v0.12m"
- board text removed: "(c) 2019 Jochen Buur"
- board text removed: "APEDSK99 v0.12l"

Commit message: update
update
Parts:
- R1, R2, R3, R4: footprint Resistor_THT:R_Axial_DIN0204_L3.6mm_D1.6mm_P5.08mm_Horizontal -> Resistor_THT:R_Axial_DIN0204_L3.6mm_D1.6mm_P5.08mm_Vertical
