File: KiCAD/APEDSK-AU.kicad_pcb (KiCad board)
At the start: 4 copper layers, 71.1 x 68.6 mm, 26 parts, among them J1 240-44-44Pins, P1 Power, P2 Analog, P3 Digital, P4 Digital, U1 74LS245, U2 74LS541, U3 74LS541, U4 GAL16V8, U5 74HC595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

Commit message: schematic cleanup
Other:
- board text added: "74HCT541"
- board text added: "74LS245"
- board text removed: "74HCT595"
- board text removed: "74LS/HCT245"
- board text removed: "74LS/HCT541"
