File: KiCAD/_autosave-APEDSK-AU.sch (KiCad schematic (older format))
At the start: 25 parts, among them J1 240-44-44Pins, P1 Power, P2 Analog, P3 Digital, P4 Digital, U1 74LS245, U2 74LS541, U3 74LS541, U4 74LS138, U5 74HC595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

Commit message: update
update
Parts:
- R1, R2, R3, R4: footprint Resistor_THT:R_Axial_DIN0204_L3.6mm_D1.6mm_P5.08mm_Horizontal -> Resistor_THT:R_Axial_DIN0204_L3.6mm_D1.6mm_P5.08mm_Vertical
Changed lines of the file:
@@
 F 0 "R1" H 8768 3396 50  0000 L CNN
 F 1 "5.1K" H 8768 3305 50  0000 L CNN
-F 2 "Resistor_THT:R_Axial_DIN0204_L3.6mm_D1.6mm_P5.08mm_Horizontal" H 8700 3350 50  0001 C CNN
+F 2 "Resistor_THT:R_Axial_DIN0204_L3.6mm_D1.6mm_P5.08mm_Vertical" H 8700 3350 50  0001 C CNN
 F 3 "~" H 8700 3350 50  0001 C CNN
 	1    8700 3350
@@
 F 0 "R2" H 9068 3496 50  0000 L CNN
 F 1 "5.1K" H 9068 3405 50  0000 L CNN
-F 2 "Resistor_THT:R_Axial_DIN0204_L3.6mm_D1.6mm_P5.08mm_Horizontal" H 9000 3450 50  0001 C CNN
+F 2 "Resistor_THT:R_Axial_DIN0204_L3.6mm_D1.6mm_P5.08mm_Vertical" H 9000 3450 50  0001 C CNN
 F 3 "~" H 9000 3450 50  0001 C CNN
 	1    9000 3450
@@
 F 0 "R3" H 9368 3496 50  0000 L CNN
 F 1 "5.1K" H 9368 3405 50  0000 L CNN
-F 2 "Resistor_THT:R_Axial_DIN0204_L3.6mm_D1.6mm_P5.08mm_Horizontal" H 9300 3450 50  0001 C CNN
+F 2 "Resistor_THT:R_Axial_DIN0204_L3.6mm_D1.6mm_P5.08mm_Vertical" H 9300 3450 50  0001 C CNN
 F 3 "~" H 9300 3450 50  0001 C CNN
 	1    9300 3450
@@
 F 0 "R4" H 9718 3396 50  0000 L CNN
 F 1 "68R" H 9718 3305 50  0000 L CNN
-F 2 "Resistor_THT:R_Axial_DIN0204_L3.6mm_D1.6mm_P5.08mm_Horizontal" H 9650 3350 50  0001 C CNN
+F 2 "Resistor_THT:R_Axial_DIN0204_L3.6mm_D1.6mm_P5.08mm_Vertical" H 9650 3350 50  0001 C CNN
 F 3 "~" H 9650 3350 50  0001 C CNN
 	1    9650 3350
