File: KiCAD/APEDSK-AU.kicad_sch (KiCad schematic)
At the start: 26 parts, among them J1 240-44-44Pins, P1 Power, P2 Analog, P3 Digital, P4 Digital, U1 74LS245, U2 74LS541, U3 74LS541, U4 GAL16V8, U5 74HC595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

Commit message: schematic cleanup
Parts:
- P3: footprint Socket_Arduino_Uno:Socket_Strip_Arduino_1x10 -> (none)
- U2, U3: value 74LS541 -> 74HCT541
Other:
- note removed: "1"
